File: battery/hardware/Schematics_batterie/Schematics_batterie.kicad_pcb (KiCad board)
At the start: 2 copper layers, 45 x 45 mm, 47 parts, among them IC1 BQ25185DLHR, J1 USB_C_Receptacle_USB2.0_16P, J2 Conn_01x02, J3 Conn_01x02, J4 Conn_ST_STDC14, J5 Conn_01x02, U1 BU33SD5WG-TR, U2 STM32G431KBTx, U3 USBLC6-2SC6

Commit message: Commencer la programmation
Routing:
- net NRST: track 19.6 -> 19.0 mm
Changed lines of the file:
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@@
+	)
+	(segment
+		(start 118.825 70.725)
+		(end 118.55 70.725)
+		(width 0.4)
+		(layer "F.Cu")
+		(net 2)
 	)
 	(segment
 		(start 130.58 74.495)
 		(end 130.75 74.325)
-		(width 0.4)
-		(layer "F.Cu")
-		(net 2)
-	)
-	(segment
-		(start 118.2 71.075)
-		(end 116.725 72.55)
 		(width 0.4)
 		(layer "F.Cu")
@@
 	)
 	(segment
-		(start 117.35 73.55)
-		(end 117.6 73.8)
-		(width 0.4)
-		(layer "F.Cu")
-		(net 2)
-	)
-	(segment
 		(start 129.3 78.425)
 		(end 129.3 79.2)
@@
 	)
 	(segment
-		(start 118.825 70.8)
-		(end 118.825 71.075)
-		(width 0.4)
-		(layer "F.Cu")
-		(net 2)
-	)
-	(segment
-		(start 118.825 71.075)
-		(end 118.2 71.075)
-		(width 0.4)
-		(layer "F.Cu")
-		(net 2)
-	)
-	(segment
 		(start 117.6 73.8)
 		(end 117.6 73.425)
@@
 		(start 132.8125 59.3)
 		(end 133.95 59.3)
+		(width 0.4)
+		(layer "F.Cu")
+		(net 2)
+	)
+	(segment
+		(start 118.55 70.725)
+		(end 116.725 72.55)
 		(width 0.4)
 		(layer "F.Cu")
@@
 	)
 	(segment
+		(start 115.39 67.54)
+		(end 115.6 67.75)
+		(width 0.3)
+		(layer "F.Cu")
+		(net 7)
+	)
+	(segment
+		(start 114.625 70.455)
+		(end 114.625 73.125)
+		(width 0.3)
+		(layer "F.Cu")
+		(net 7)
+	)
+	(segment
+		(start 120.725 75.85)
+		(end 122.525 74.05)
+		(width 0.3)
+		(layer "F.Cu")
+		(net 7)
+	)
+	(segment
+		(start 122.6 74.0375)
+		(end 122.6125 74.05)
+		(width 0.3)
+		(layer "F.Cu")
+		(net 7)
+	)
+	(segment
+		(start 114.625 73.125)
+		(end 117.35 75.85)
+		(width 0.3)
+		(layer "F.Cu")
+		(net 7)
+	)
+	(segment
+		(start 122.6 72.175)
+		(end 122.6 74.0375)
+		(width 0.3)
+		(layer "F.Cu")
+		(net 7)
+	)
+	(segment
+		(start 117.35 75.85)
+		(end 120.725 75.85)
+		(width 0.3)
+		(layer "F.Cu")
+		(net 7)
+	)
+	(segment
 		(start 115.6 69.48)
 		(end 114.625 70.455)
@@
 	)
 	(segment
-		(start 122.6 74.0375)
-		(end 122.6125 74.05)
+		(start 114.1 67.54)
+		(end 115.39 67.54)
 		(width 0.3)
 		(layer "F.Cu")
@@
 	)
 	(segment
-		(start 122.6 72.175)
-		(end 122.6 74.0375)
-		(width 0.3)
-		(layer "F.Cu")
-		(net 7)
-	)
-	(segment
-		(start 114.1 67.54)
-		(end 114.93 67.54)
-		(width 0.3)
-		(layer "F.Cu")
-		(net 7)
-	)
-	(segment
-		(start 114.625 67.845)
-		(end 114.625 68.14)
-		(width 0.3)
-		(layer "F.Cu")
-		(net 7)
-	)
-	(segment
-		(start 114.625 70.455)
-		(end 114.625 73.125)
-		(width 0.3)
-		(layer "F.Cu")
-		(net 7)
-	)
-	(segment
-		(start 117.35 75.85)
-		(end 120.725 75.85)
-		(width 0.3)
-		(layer "F.Cu")
-		(net 7)
-	)
-	(segment
-		(start 114.625 68.14)
-		(end 115.6 68.14)
-		(width 0.3)
-		(layer "F.Cu")
-		(net 7)
-	)
-	(segment
-		(start 114.625 73.125)
-		(end 117.35 75.85)
-		(width 0.3)
-		(layer "F.Cu")
-		(net 7)
-	)
-	(segment
-		(start 114.93 67.54)
-		(end 114.625 67.845)
-		(width 0.3)
-		(layer "F.Cu")
-		(net 7)
-	)
-	(segment
-		(start 115.6 68.14)
+		(start 115.6 67.75)
 		(end 115.6 69.48)
 		(width 0.3)
 		(layer "F.Cu")
-		(net 7)
-	)
-	(segment
-		(start 120.725 75.85)
-		(end 122.525 74.05)
-		(width 0.3)
-		(layer "F.Cu")
