File: LED/veste lumineuse_LEDS/Hardware/veste lumineuse_LEDS.kicad_sch (KiCad schematic)
At the start: 2 parts, among them U1 STM32G431KBTx, U2 CH224K

Commit message: schema kicad 10_03_25 1
Parts:
- removed U2: CH224K, Package_SO:SSOP-10-1EP_3.9x4.9mm_P1mm_EP2.1x3.3mm, symbol Interface_USB:CH224K
- added C3, C4, C5, C9: 100n, FootprintGamelGe2_v8.0:C_Rect_L7.0mm_W2.5mm_P5.00mm, symbol SymbGamelGe2_v8.0:C
- added C6: 4.7µ, FootprintGamelGe2_v8.0:C_Rect_L7.0mm_W2.5mm_P5.00mm, symbol SymbGamelGe2_v8.0:C
- added C7, C8: 0.47µ, FootprintGamelGe2_v8.0:C_Rect_L7.0mm_W2.5mm_P5.00mm, symbol SymbGamelGe2_v8.0:C
- added D2, D3: LED, LED_SMD:LED_0201_0603Metric, symbol Device:LED
- added J2: Conn_ST_STDC14, symbol Connector:Conn_ST_STDC14
- added J3: Omnimate2, FootprintGamelGe2_v8.0:OmnimateSL-5,08_1x02_P5.08mm_Vertical, symbol SymbGamelGe2_v8.0:Omnimate2
- added R1, R2: 1k, FootprintGamelGe2_v8.0:R_Axial_DIN0207_L6.3mm_D2.5mm_P10.16mm_Horizontal, symbol SymbGamelGe2_v8.0:R
- added U3: BU33SD5WG-TR, Package_TO_SOT_SMD:SOT-23-5, symbol Regulator_Linear:MCP1802x-xx02xOT
Connections:
- net +3.3V: now reaches U1.1 (VDD)
- net +3.3V: now also U1.15 (VDDA), U1.17 (VDD), C3.1, C4.1, C5.1, C6.1, C8.1, D3.2 (A), J2.3 (VCC), U3.5 (VOUT)
- net GND: now reaches U1.14 (VSSA)
- net GND: now also U1.16 (VSS), U1.32 (VSS), C3.2, C4.2, C5.2, C6.2, C7.2, C8.2, C9.1, J2.11 (GNDDetect), J2.5 (GND), J2.7 (GND), J3.1 (Pin_1), R1.2, R2.2, U3.2 (GND)
- net VCP_TX: now reaches U1.19 (PA9)
- net VCP_TX: now also J2.14 (VCP_TX)
- net VCP_RX: now reaches U1.20 (PA10)
- net VCP_RX: now also J2.13 (VCP_RX)
- net SWDIO: now reaches U1.23 (PA13)
- net SWDIO: now also J2.4 (JTMS/SWDIO)
- net SWCLK: now reaches U1.24 (PA14)
- net SWCLK: now also J2.6 (JCLK/SWCLK)
- net RST: now reaches U1.4 (PG10)
- net RST: now also C9.2, J2.12 (~{RST})
- net at U1.6 (PA1): now also D2.2 (A)
- net MIDI_TX: now reaches U1.7 (PA2)
- net MIDI_RX: now reaches U1.8 (PA3)
- new net: D2.1 (K), R1.1
- new net: D3.1 (K), R2.1
- new net +5V: C7.1, J3.2 (Pin_2), U3.1 (VIN), U3.3 (~{SHDN})
- no-connect marks 0 -> 21
Other:
- moved on the sheet: U1

Commit message: schema final 10_03_25
Parts:
- removed J2: Conn_ST_STDC14, symbol Connector:Conn_ST_STDC14
- added J1: Conn_ST_STDC14, Connector_PinHeader_1.27mm:PinHeader_2x07_P1.27mm_Vertical_SMD, symbol Connector:Conn_ST_STDC14
- C3, C4, C5, C6, C7, C8, C9: footprint FootprintGamelGe2_v8.0:C_Rect_L7.0mm_W2.5mm_P5.00mm -> Capacitor_SMD:C_0402_1005Metric
- D2, D3: footprint LED_SMD:LED_0201_0603Metric -> LED_SMD:LED_0402_1005Metric
- R1, R2: footprint FootprintGamelGe2_v8.0:R_Axial_DIN0207_L6.3mm_D2.5mm_P10.16mm_Horizontal -> Resistor_SMD:R_0402_1005Metric
Connections:
- net +3.3V: now also J1.3 (VCC)
- net GND: now also J1.11 (GNDDetect), J1.5 (GND), J1.7 (GND)
- net RST: now also J1.12 (~{RST})
- net SWCLK: now also J1.6 (JCLK/SWCLK)
- net SWDIO: now also J1.4 (JTMS/SWDIO)
- net VCP_RX: now also J1.13 (VCP_RX)
- net VCP_TX: now also J1.14 (VCP_TX)

Commit message: fin schema 10_03_25
Parts:
- removed J3: Omnimate2, FootprintGamelGe2_v8.0:OmnimateSL-5,08_1x02_P5.08mm_Vertical, symbol SymbGamelGe2_v8.0:Omnimate2
- added J2: Conn_01x02, Connector_JST:JST_XH_B2B-XH-A_1x02_P2.50mm_Vertical, symbol Connector_Generic:Conn_01x02
- added J3: Conn_01x03, Connector_JST:JST_XH_B3B-XH-A_1x03_P2.50mm_Vertical, symbol Connector_Generic:Conn_01x03
- D2, D3: footprint LED_SMD:LED_0402_1005Metric -> LED_SMD:LED_0603_1608Metric
Connections:
- net +5V: now also J2.2 (Pin_2), J3.3 (Pin_3)
- net GND: now also J2.1 (Pin_1), J3.1 (Pin_1)
Changed lines of the file:
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@@
+	(wire
+		(pts
+			(xy 50.8 85.09) (xy 53.34 85.09)
+		)
+		(stroke
+			(width 0)
+			(type default)
+		)
+	)
 	(wire
 		(pts
@@
 		(pts
 			(xy 217.17 46.99) (xy 217.17 49.53)
+		)
+		(stroke
+			(width 0)
+			(type default)
+		)
+	)
+	(wire
+		(pts
+			(xy 53.34 85.09) (xy 53.34 83.82)
 		)
 		(stroke
@@
 			)
 		)
-		(property "Footprint" "LED_SMD:LED_0402_1005Metric"
+		(property "Footprint" "LED_SMD:LED_0603_1608Metric"
 			(at 234.95 73.66 0)
 			(effects
@@
 	)
 	(symbol
+		(lib_id "Connector_Generic:Conn_01x02")
+		(at 27.94 44.45 180)
+		(unit 1)
+		(exclude_from_sim no)
+		(in_bom yes)
+		(on_board yes)
+		(dnp no)
+		(fields_autoplaced yes)
+		(property "Reference" "J2"
+			(at 27.94 35.56 0)
+			(effects
+				(font
+					(size 1.27 1.27)
+				)
+			)
+		)
+		(property "Value" "Conn_01x02"
+			(at 27.94 38.1 0)
+			(effects
+				(font
+					(size 1.27 1.27)
+				)
+			)
+		)
+		(property "Footprint" "Connector_JST:JST_XH_B2B-XH-A_1x02_P2.50mm_Vertical"
+			(at 27.94 44.45 0)
+			(effects
+				(font
+					(size 1.27 1.27)
+				)
+				(hide yes)
+			)
+		)
+		(property "Datasheet" "~"
+			(at 27.94 44.45 0)
+			(effects
+				(font
+					(size 1.27 1.27)
+				)
+				(hide yes)
+			)
+		)
+		(property "Description" "Generic connector, single row, 01x02, script generated (kicad-library-utils/schlib/autogen/connector/)"
+			(at 27.94 44.45 0)
+			(effects
+				(font
+					(size 1.27 1.27)
+				)
+				(hide yes)
+			)
+		)
+		(pin "2"
+		)
+		(pin "1"
+		)
+		(instances
+			(project ""
+				(path "/67146bde-f542-429a-9136-9c8458814419"
+					(reference "J2")
+					(unit 1)
+				)
+			)
+		)
+	)
+	(symbol
 		(lib_id "Regulator_Linear:MCP1802x-xx02xOT")
 		(at 71.12 41.91 0)
@@
 	)
 	(symbol
+		(lib_id "power:GND")
+		(at 50.8 90.17 0)
+		(unit 1)
+		(exclude_from_sim no)
+		(in_bom yes)
+		(on_board yes)
+		(dnp no)
+		(fields_autoplaced yes)
+		(property "Reference" "#PWR016"
+			(at 50.8 96.52 0)
+			(effects
+				(font
+					(size 1.27 1.27)
+				)
+				(hide yes)
+			)
+		)
+		(property "Value" "GND"
+			(at 50.8 95.25 0)
+			(effects
+				(font
+					(size 1.27 1.27)
+				)
+			)
+		)
+		(property "Footprint" ""
+			(at 50.8 90.17 0)
+			(effects
+				(font
+					(size 1.27 1.27)
+				)
+				(hide yes)
+			)
+		)
+		(property "Datasheet" ""
+			(at 50.8 90.17 0)
+			(effects
+				(font
+					(size 1.27 1.27)
+				)
+				(hide yes)
+			)
+		)
+		(property "Description" "Power symbol creates a global label with name \"GND\" , ground"
+			(at 50.8 90.17 0)
+			(effects
+				(font
+					(size 1.27 1.27)
+				)
+				(hide yes)
+			)
+		)
+		(pin "1"
+		)
+		(instances
+			(project "veste lumineuse_LEDS"
+				(path "/67146bde-f542-429a-9136-9c8458814419"
+					(reference "#PWR016")
+					(unit 1)
+				)
+			)
+		)
+	)
+	(symbol
 		(lib_id "power:+5V")
 		(at 43.18 35.56 0)
@@
 	)
 	(symbol
-		(lib_id "SymbGamelGe2_v8.0:Omnimate2")
-		(at 27.94 41.91 0)
+		(lib_id "power:+5V")
+		(at 53.34 83.82 0)
+		(unit 1)
+		(exclude_from_sim no)
+		(in_bom yes)
+		(on_board yes)
+		(dnp no)
+		(property "Reference" "#PWR015"
+			(at 53.34 87.63 0)
+			(effects
+				(font
+					(size 1.27 1.27)
+				)
+				(hide yes)
+			)
+		)
+		(property "Value" "+5V"
+			(at 53.848 84.328 0)
+			(effects
+				(font
+					(size 1.27 1.27)
+				)
+				(justify left)
+			)
+		)
+		(property "Footprint" ""
+			(at 53.34 83.82 0)
+			(effects
+				(font
+					(size 1.27 1.27)
+				)
+				(hide yes)
+			)
+		)
+		(property "Datasheet" ""
+			(at 53.34 83.82 0)
+			(effects
+				(font
+					(size 1.27 1.27)
+				)
+				(hide yes)
+			)
+		)
+		(property "Description" "Power symbol creates a global label with name \"+5V\""
+			(at 53.34 83.82 0)
+			(effects
+				(font
+					(size 1.27 1.27)
+				)
+				(hide yes)
+			)
+		)
+		(pin "1"
+		)
+		(instances
+			(project "veste lumineuse_LEDS"
+				(path "/67146bde-f542-429a-9136-9c8458814419"
+					(reference "#PWR015")
+					(unit 1)
+				)
+			)
+		)
+	)
+	(symbol
+		(lib_id "Connector_Generic:Conn_01x03")
+		(at 45.72 87.63 180)
 		(unit 1)
 		(exclude_from_sim no)
@@
 		(fields_autoplaced yes)
 		(property "Reference" "J3"
-			(at 28.3252 33.02 0)
-			(effects
-				(font
-					(size 1.27 1.27)
-				)
-			)
-		)
-		(property "Value" "Omnimate2"
-			(at 28.3252 35.56 0)
-			(effects
-				(font
-					(size 1.27 1.27)
-				)
-			)
-		)
-		(property "Footprint" "FootprintGamelGe2_v8.0:OmnimateSL-5,08_1x02_P5.08mm_Vertical"
-			(at 29.21 41.91 0)
+			(at 45.72 78.74 0)
+			(effects
+				(font
+					(size 1.27 1.27)
+				)
+			)
+		)
+		(property "Value" "Conn_01x03"
+			(at 45.72 81.28 0)
+			(effects
+				(font
+					(size 1.27 1.27)
+				)
+			)
+		)
+		(property "Footprint" "Connector_JST:JST_XH_B3B-XH-A_1x03_P2.50mm_Vertical"
+			(at 45.72 87.63 0)
 			(effects
 				(font
@@
 		)
 		(property "Datasheet" "~"
-			(at 29.21 41.91 0)
-			(effects
-				(font
-					(size 1.27 1.27)
-				)
-				(hide yes)
-			)
-		)
-		(property "Description" "Connector BL/SL 5.08, single row, 01x02, power supply connector"
-			(at 27.94 41.91 0)
-			(effects
-				(font
-					(size 1.27 1.27)
-				)
-				(hide yes)
-			)
+			(at 45.72 87.63 0)
+			(effects
+				(font
+					(size 1.27 1.27)
+				)
+				(hide yes)
+			)
+		)
+		(property "Description" "Generic connector, single row, 01x03, script generated (kicad-library-utils/schlib/autogen/connector/)"
+			(at 45.72 87.63 0)
+			(effects
+				(font
+					(size 1.27 1.27)
+				)
+				(hide yes)
+			)
+		)
+		(pin "3"
 		)
 		(pin "1"
@@
 			)
 		)
-		(property "Footprint" "LED_SMD:LED_0402_1005Metric"
+		(property "Footprint" "LED_SMD:LED_0603_1608Metric"
 			(at 104.14 39.37 0)
 			(effects
