File: LED/veste lumineuse_LEDS/Hardware/_autosave-veste lumineuse_LEDS.kicad_sch (KiCad schematic)
At the start: 22 parts, among them J1 Conn_ST_STDC14, J2 Conn_01x02, J3 LED NEOPIXEL, J4 MIDI UART, U1 STM32G431KBTx, U3 BU33SD5WG-TR

Commit message: fin schema/root 31-03-2025
Parts:
- J2: value Conn_01x02 -> BATTERY
Changed lines of the file:
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@@
 			)
 		)
-		(property "Value" "Conn_01x02"
+		(property "Value" "BATTERY"
 			(at 27.94 38.1 0)
 			(effects
