File: LED/veste lumineuse_LEDS/Hardware/veste lumineuse_LEDS.kicad_pcb (KiCad board)
At the start: 2 copper layers, 14 parts, among them J3 Omnimate2, U1 STM32G431KBTx, U3 BU33SD5WG-TR

Commit message: schema final 10_03_25
Parts:
- added J1: Conn_ST_STDC14, Connector_PinHeader_1.27mm:PinHeader_2x07_P1.27mm_Vertical_SMD, F.Cu at (84.5, 51.0)
- C3, C4, C5, C6, C7, C8, C9: footprint FootprintGamelGe2_v8.0:C_Rect_L7.0mm_W2.5mm_P5.00mm -> Capacitor_SMD:C_0402_1005Metric
- D2, D3: footprint LED_SMD:LED_0201_0603Metric -> LED_SMD:LED_0402_1005Metric
- R1, R2: footprint FootprintGamelGe2_v8.0:R_Axial_DIN0207_L6.3mm_D2.5mm_P10.16mm_Horizontal -> Resistor_SMD:R_0402_1005Metric
- moved C7 42.5 mm to (47.9, 56.1), turned to 90 degrees
- moved J3 39.5 mm to (36.0, 58.0), turned to 90 degrees
- moved D2 37.4 mm to (68.0, 84.0)
- moved C8 36.5 mm to (60.5, 54.5)
- moved C3 35.9 mm to (51.0, 48.0), turned to 90 degrees
- moved C4 35.1 mm to (54.0, 48.0), turned to 90 degrees
- moved C5 35.0 mm to (57.0, 48.0), turned to 90 degrees
- moved C6 35.0 mm to (61.0, 48.0), turned to 90 degrees
- moved R1 32.6 mm to (67.0, 86.5), turned to 180 degrees
- moved U3 29.3 mm to (55.5, 55.5)
- moved D3 28.4 mm to (60.5, 56.0), turned to 180 degrees
- moved C9 18.5 mm to (66.0, 82.5)
- moved R2 10.00 mm to (60.5, 58.5), turned to 180 degrees
Connections:
- U1 pad 14: unconnected-(U1-VSSA-Pad14) -> GND
- U1 pad 16: unconnected-(U1-VSS-Pad16) -> GND
- U1 pad 19: TX -> VCP_TX
- U1 pad 20: RX -> VCP_RX
- U1 pad 32: unconnected-(U1-VSS-Pad16)_1 -> GND
- U1 pad 7: unconnected-(U1-PA2-Pad7) -> MIDI_TX
- U1 pad 8: unconnected-(U1-PA3-Pad8) -> MIDI_RX

Commit message: fin schema/root 31-03-2025
Parts:
- added H1: MountingHole_Pad, MountingHole:MountingHole_3.2mm_M3_Pad_Via, F.Cu at (130.0, 100.0)
- added H2: MountingHole_Pad, MountingHole:MountingHole_3.2mm_M3_Pad_Via, F.Cu at (170.0, 100.0)
- added H3: MountingHole_Pad, MountingHole:MountingHole_3.2mm_M3_Pad_Via, F.Cu at (170.0, 120.0)
- added H4: MountingHole_Pad, MountingHole:MountingHole_3.2mm_M3_Pad_Via, F.Cu at (130.0, 120.0)
- added J2: BATTERY, Connector_JST:JST_XH_B2B-XH-A_1x02_P2.50mm_Vertical, F.Cu at (130.0, 112.0)
- added J4: MIDI UART, Connector_JST:JST_XH_B3B-XH-A_1x03_P2.50mm_Vertical, F.Cu at (153.0, 100.0)
- added TP1: 3.3V, TestPoint:TestPoint_Pad_D2.0mm, F.Cu at (159.5, 119.8)
- C6: footprint Capacitor_SMD:C_0402_1005Metric -> Capacitor_SMD:C_0603_1608Metric
- C7, C8: value 0.47µ -> 1u; footprint Capacitor_SMD:C_0402_1005Metric -> Capacitor_SMD:C_0603_1608Metric
- D2, D3: footprint LED_SMD:LED_0402_1005Metric -> LED_SMD:LED_0603_1608Metric
- J3: value Omnimate2 -> LED NEOPIXEL; footprint FootprintGamelGe2_v8.0:OmnimateSL-5,08_1x02_P5.08mm_Vertical -> Connector_JST:JST_XH_B3B-XH-A_1x03_P2.50mm_Vertical
- moved C4 123.2 mm to (156.0, 117.0), turned to -135 degrees
- moved C5 118.4 mm to (152.5, 118.0), turned to 180 degrees
- moved C6 116.1 mm to (152.5, 119.5), turned to 180 degrees
- moved J3 112.2 mm to (140.0, 100.0), turned to 0 degrees
- moved C3 111.8 mm to (146.0, 107.0), turned to 45 degrees
- moved C7 106.0 mm to (137.0, 113.5), turned to 180 degrees
- moved U3 98.3 mm to (137.0, 110.5), turned to 90 degrees
- moved J1 98.2 mm to (163.0, 110.0), turned to 180 degrees
- moved R2 96.7 mm to (140.0, 113.5), turned to -90 degrees
- moved D3 96.4 mm to (140.0, 110.5), turned to 90 degrees
- moved C8 93.1 mm to (137.0, 107.5)
- moved C9 83.7 mm to (144.5, 111.5)
- moved U1 81.7 mm to (151.0, 112.0)
- moved R1 81.5 mm to (143.5, 114.5), turned to 0 degrees
- moved D2 81.1 mm to (143.8, 113.0)
Connections:
- net Net-(D2-A) renamed /LED_STATUS
- C7 pad 1: +5V -> GND
- C7 pad 2: GND -> +5V
- J3 pad 2: +5V -> LED_NP
- U1 pad 18: unconnected-(U1-PA8-Pad18) -> LED_NP
- U1 pad 31: unconnected-(U1-PB8-Pad31) -> GND
Routing:
- net +3.3V: track 0.00 -> 54.0 mm
- net +5V: track 0.00 -> 34.0 mm
- net LED_NP: track 0.00 -> 30.0 mm, vias 0 -> 4
- net MIDI_TX: track 0.00 -> 20.5 mm, vias 0 -> 2
- net MIDI_RX: track 0.00 -> 19.8 mm, vias 0 -> 2
- net GND: track 0.00 -> 18.4 mm, vias 0 -> 52
- net RST: track 0.00 -> 17.8 mm, vias 0 -> 2
- net VCP_RX: track 0.00 -> 17.4 mm, vias 0 -> 2
- net VCP_TX: track 0.00 -> 11.7 mm, vias 0 -> 2
- net SWDIO: track 0.00 -> 6.93 mm
- net SWCLK: track 0.00 -> 6.73 mm
- net /LED_STATUS: track 0.00 -> 2.33 mm
- net Net-(D3-K): track 0.00 -> 1.70 mm
- net Net-(D2-K): track 0.00 -> 1.50 mm
- added copper zone on B.Cu, net GND
- added copper zone on F.Cu, net GND
Other:
- board outline added: 48 x 28 mm
- board text added: "+"
- board text added: "-"
- board text added: "BATT"
- board text added: "LED"
- board text added: "MIDI"
